File: Hardware/AcrylicBadge.kicad_sch (KiCad schematic)
At the start: 55 parts, among them J1 CellP, J2 CellN, J3 Conn_02x03_Odd_Even, J4 USB4125-GF-A, U1 ATmega328PB-AU, U2 PAM2401SCADJ, U3 MCP73833T-AMI/UN, U4 BQ29737, U5 CSD16406Q3, U6 CSD16406Q3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

Commit message: Started PCB Layout
Parts:
- Y1: footprint Crystal:Crystal_SMD_HC49-SD_HandSoldering -> Crystal:Crystal_SMD_HC49-SD
Changed lines of the file:
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@@
 			)
 		)
-		(property "Footprint" "Crystal:Crystal_SMD_HC49-SD_HandSoldering"
+		(property "Footprint" "Crystal:Crystal_SMD_HC49-SD"
 			(at 72.39 49.53 0)
 			(effects
